Commit message: Fixed some tfs and added launch to run in phisical robot(lidar 3d and kobuki)

File: uvone_robot_description/urdf/include/astra.urdf.xacro (robot description, xacro)
@@ -41,6 +41,6 @@
     <xacro:macro name="sensor_astra" params="parent posz">
         <joint name="camera_rgb_joint" type="fixed">
-        <origin xyz="0.012 0 ${posz}"
-                rpy="0 0.30 0"/>
+        <origin xyz="0.012 -0.070 ${posz}"
+                rpy="0 0.37 0"/>
         <parent link="${parent}"/>
         <child link="camera_rgb_frame" />
@@ -48,5 +48,5 @@
         <link name="camera_rgb_frame"/>
         <joint name="camera_rgb_optical_joint" type="fixed">
-        <origin xyz="0 0.014 0" rpy="${-M_PI/2} 0 ${-M_PI/2}" />
+        <origin xyz="0 -0.014 0" rpy="${-M_PI/2} 0 ${-M_PI/2}" />
         <parent link="camera_rgb_frame" />
         <child link="camera_rgb_optical_frame" />
@@ -54,5 +54,5 @@
         <link name="camera_rgb_optical_frame"/>
         <joint name="camera_depth_joint" type="fixed">
-        <origin xyz="0 -0.035 0" rpy="0 0 0" /><!-- ha cambiado !! posy-->
+        <origin xyz="0 -0.036 0" rpy="0 0 0" /><!-- ha cambiado !! posy-->
         <parent link="camera_rgb_frame" />
         <child link="camera_depth_frame" />

File: uvone_robot_description/urdf/model.urdf.xacro (robot description, xacro)
@@ -33,4 +33,4 @@
   </link>
   <!-- Camara astra -->
-  <xacro:sensor_astra parent="base_link" posz="1.358"/>  <!-- Primer escalon: posz=0.718 --> <!-- Segundo escalon: posz=1.358 -->
+  <xacro:sensor_astra parent="base_link" posz="1.238"/>  <!-- Primer escalon: posz=0.718 --> <!-- Segundo escalon: posz=1.358 -->
 </robot>
